File: Hardware/电源模块.kicad_sch (KiCad schematic)
At the start: 0 parts

Commit message: 完成电源模块电路原理图
Parts:
- added C10, C12, C14, C16, C18, C19, C23, C5, C8: 104, symbol Device:C
- added C11, C13, C15, C6, C7, C9: 10uF, symbol Device:C
- added C17, C22: 22uF, symbol Device:C
- added C20: 1nF, symbol Device:C
- added C21: 33pF, symbol Device:C
- added J1: Barrel_Jack_Switch, symbol Connector:Barrel_Jack_Switch
- added L1: 5.5uH, symbol Device:L
- added R10: 75K, symbol Device:R
- added R11: 40.2K, symbol Device:R
- added R12: 0, symbol Device:R
- added R13: 20K, symbol Device:R
- added R14: 7.5K, symbol Device:R
- added R15: 20, symbol Device:R
- added R9: 100K, symbol Device:R
- added SW5: ~, Switching_Devices:Self_Locking_Switch_5.8_5.8, symbol Switching_Devices:Self_Locking_Switch
- added U5: AMS1117-1.8, Package_TO_SOT_SMD:SOT-223-3_TabPin2, symbol Regulator_Linear:AMS1117-1.8
- added U6: AMS1117-2.5, Package_TO_SOT_SMD:SOT-223-3_TabPin2, symbol Regulator_Linear:AMS1117-2.5
- added U7: AMS1117-3.3, Package_TO_SOT_SMD:SOT-223-3_TabPin2, symbol Regulator_Linear:AMS1117-3.3
- added U8: MP2315GJ, Package_TO_SOT_SMD:TSOT-23-8, symbol My_Converter_DCDC:MP2315GJ
Connections:
- new net: R13.1, U8.8 (FB)
- new net: R11.2, R12.2, R13.2, R14.1
- new net: J1.1, SW5.2, SW5.5
- new net: C21.2, R12.1
- new net: C23.2, L1.2, U8.3 (SW)
- new net: C23.1, R15.1
- new net: C19.1, U8.7 (VCC)
- new net: C20.2, R10.2, U8.1 (AAM)
- new net: R15.2, U8.5 (BST)
- new net: R9.1, U8.6 (EN/SYNC)
- new net +12V: C17.1, C18.1, R9.2, SW5.3, SW5.4, U8.2 (IN)
- new net +1V8: C7.1, C8.1, U5.2 (VO)
- new net +2V5: C11.1, C12.1, U6.2 (VO)
- new net +3.3V: C13.1, C14.1, U7.2 (VO)
- new net +5V: C10.1, C15.1, C16.1, C21.1, C22.1, C5.1, C6.1, C9.1, L1.1, R11.1, U5.3 (VI), U6.3 (VI), U7.3 (VI)
- new net GND: C10.2, C11.2, C12.2, C13.2, C14.2, C15.2, C16.2, C17.2, C18.2, C19.2, C20.1, C22.2, C5.2, C6.2, C7.2, C8.2, C9.2, J1.2, J1.3, R10.1, R14.2, U5.1 (GND), U6.1 (GND), U7.1 (GND), U8.4 (GND)
- no-connect marks 0 -> 2

Commit message: 2023/3/29
Parts:
- removed C17: 22uF, symbol Device:C
- removed SW5: ~, Switching_Devices:Self_Locking_Switch_5.8_5.8, symbol Switching_Devices:Self_Locking_Switch
- added C6: 22uF, Capacitor_SMD:CP_Elec_4x5.4, symbol Device:C_Polarized
- added SW5: ~, symbol Library:SW
- C10: renamed from C21; footprint (none) -> Capacitor_SMD:C_0402_1005Metric
- C11: renamed from C19; footprint (none) -> Capacitor_SMD:C_0402_1005Metric
- C12: renamed from C22; footprint (none) -> Capacitor_SMD:C_1206_3216Metric
- C13: renamed from C6; footprint (none) -> Capacitor_SMD:C_0603_1608Metric
- C14: renamed from C9; footprint (none) -> Capacitor_SMD:C_0603_1608Metric
- C15: footprint (none) -> Capacitor_SMD:C_0603_1608Metric
- C16: renamed from C5; footprint (none) -> Capacitor_SMD:C_0402_1005Metric
- C17: renamed from C10; footprint (none) -> Capacitor_SMD:C_0402_1005Metric
- C18: renamed from C16; footprint (none) -> Capacitor_SMD:C_0402_1005Metric
- C19: renamed from C7; footprint (none) -> Capacitor_SMD:C_0603_1608Metric
- C20: renamed from C11; footprint (none) -> Capacitor_SMD:C_0603_1608Metric
- C21: renamed from C13; footprint (none) -> Capacitor_SMD:C_0603_1608Metric
- C22: renamed from C8; footprint (none) -> Capacitor_SMD:C_0402_1005Metric
- C23: renamed from C12; footprint (none) -> Capacitor_SMD:C_0402_1005Metric
- C24: renamed from C14; footprint (none) -> Capacitor_SMD:C_0402_1005Metric
- C7: renamed from C18; footprint (none) -> Capacitor_SMD:C_0402_1005Metric
- C8: renamed from C20; footprint (none) -> Capacitor_SMD:C_0402_1005Metric
- C9: renamed from C23; footprint (none) -> Capacitor_SMD:C_0402_1005Metric
- J3: renamed from J1; footprint (none) -> Connector_BarrelJack:BarrelJack_CLIFF_FC681465S_SMT_Horizontal
- L1: footprint (none) -> Inductor_SMD:L_2512_6332Metric_Pad1.52x3.35mm_HandSolder
- R10: renamed from R9; footprint (none) -> Resistor_SMD:R_0402_1005Metric
- R11: renamed from R12; footprint (none) -> Resistor_SMD:R_0402_1005Metric
- R12: renamed from R14; footprint (none) -> Resistor_SMD:R_0402_1005Metric
- R6: renamed from R10; footprint (none) -> Resistor_SMD:R_0402_1005Metric
- R7: renamed from R15; footprint (none) -> Resistor_SMD:R_0402_1005Metric
- R8: renamed from R13; footprint (none) -> Resistor_SMD:R_0402_1005Metric
- R9: renamed from R11; footprint (none) -> Resistor_SMD:R_0402_1005Metric
- renumbered U8 to U2, U5 to U3, U6 to U4, U7 to U5
Connections:
- net +12V: now also C6.1, SW5.3
- net GND: now also C6.2
- net at J3.1: now also SW5.2
- net +3.3V renamed +3V3
- no-connect marks 2 -> 1
Other:
- moved on the sheet: C10, C11, C12, C13, C14, C15, C16, C17, C18, C19, C20, C21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
