File: Hardware/Warehouse-on-STM32.kicad_sch (KiCad schematic)
At the start: 22 parts, among them J1 ESP8266, J2 Conn_01x05, SW1 SW_Push, SW2 SW_Push, SW3 SW_Push, SW4 SW_Push, U1 STM32F103C8Tx, Y1 8MHz

Commit message: 绘制第一版
Connections:
- net SCL: now also U1.21 (PB10); no longer U1.42 (PB6)
- net SDA: now also U1.22 (PB11); no longer U1.43 (PB7)
- no-connect marks 16 -> 14
Changed lines of the file:
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@@
   (no_connect (at 237.49 54.61))
   (no_connect (at 237.49 52.07))
-  (no_connect (at 204.47 90.17))
-  (no_connect (at 204.47 87.63))
   (no_connect (at 204.47 92.71))
   (no_connect (at 204.47 64.77))
@@
     (stroke (width 0) (type default))
   )
+  (wire (pts (xy 182.88 87.63) (xy 204.47 87.63))
+    (stroke (width 0) (type default))
+  )
   (wire (pts (xy 76.2 111.76) (xy 76.2 113.03))
     (stroke (width 0) (type default))
@@
     (stroke (width 0) (type default))
   )
+  (wire (pts (xy 182.88 90.17) (xy 204.47 90.17))
+    (stroke (width 0) (type default))
+  )
   (wire (pts (xy 156.21 76.2) (xy 167.64 76.2))
     (stroke (width 0) (type default))
@@
     (stroke (width 0) (type default))
   )
-  (wire (pts (xy 182.88 80.01) (xy 204.47 80.01))
-    (stroke (width 0) (type default))
-  )
   (wire (pts (xy 156.21 86.36) (xy 156.21 87.63))
     (stroke (width 0) (type default))
@@
     (stroke (width 0) (type default))
   )
-  (wire (pts (xy 182.88 77.47) (xy 204.47 77.47))
-    (stroke (width 0) (type default))
-  )
   (wire (pts (xy 58.42 102.87) (xy 64.77 102.87))
     (stroke (width 0) (type default))
@@
     (effects (font (size 1.27 1.27)) (justify left bottom))
   )
+  (label "SCL" (at 182.88 87.63 0) (fields_autoplaced)
+    (effects (font (size 1.27 1.27)) (justify left bottom))
+  )
   (label "SDA" (at 43.18 81.28 0) (fields_autoplaced)
     (effects (font (size 1.27 1.27)) (justify left bottom))
@@
     (effects (font (size 1.27 1.27)) (justify left bottom))
   )
-  (label "SCL" (at 182.88 77.47 0) (fields_autoplaced)
-    (effects (font (size 1.27 1.27)) (justify left bottom))
-  )
   (label "APH" (at 43.18 49.53 0) (fields_autoplaced)
     (effects (font (size 1.27 1.27)) (justify left bottom))
@@
     (effects (font (size 1.27 1.27)) (justify left bottom))
   )
-  (label "SDA" (at 182.88 80.01 0) (fields_autoplaced)
-    (effects (font (size 1.27 1.27)) (justify left bottom))
-  )
   (label "ESP_RX" (at 251.46 41.91 0) (fields_autoplaced)
     (effects (font (size 1.27 1.27)) (justify left bottom))
@@
     (effects (font (size 1.27 1.27)) (justify left bottom))
   )
+  (label "SDA" (at 182.88 90.17 0) (fields_autoplaced)
+    (effects (font (size 1.27 1.27)) (justify left bottom))
+  )
