File: Hardware/驱动模块.kicad_sch (KiCad schematic)
At the start: 0 parts

Commit message: 完成电源模块电路原理图
Parts:
- added J2, J3, J4, J5: Conn_01x02_Socket, symbol Connector:Conn_01x02_Socket
- added U10, U9: TB6612FNG, Package_SO:SSOP-24_5.3x8.2mm_P0.65mm, symbol Driver_Motor:TB6612FNG
Connections:
- new net: J5.1 (Pin_1), U10.11 (BO1), U10.12 (BO1)
- new net: J5.2 (Pin_2), U10.7 (BO2), U10.8 (BO2)
- new net: J2.1 (Pin_1), U9.1 (AO1), U9.2 (AO1)
- new net: J2.2 (Pin_2), U9.5 (AO2), U9.6 (AO2)
- new net: J4.1 (Pin_1), U10.1 (AO1), U10.2 (AO1)
- new net: J4.2 (Pin_2), U10.5 (AO2), U10.6 (AO2)
- new net: J3.1 (Pin_1), U9.11 (BO1), U9.12 (BO1)
- new net: J3.2 (Pin_2), U9.7 (BO2), U9.8 (BO2)
- new net +12V: U10.13 (VM2), U10.14 (VM3), U10.24 (VM1), U9.13 (VM2), U9.14 (VM3), U9.24 (VM1)
- new net +3.3V: U10.20 (VCC), U9.20 (VCC)
- new net GND: U10.10 (PGND2), U10.18 (GND), U10.3 (PGND1), U10.4 (PGND1), U10.9 (PGND2), U9.10 (PGND2), U9.18 (GND), U9.3 (PGND1), U9.4 (PGND1), U9.9 (PGND2)

Commit message: 运行DRC前
Connections:
- net PWMB1: now reaches U10.15 (PWMB)
- net BIN21: now reaches U10.16 (BIN2)
- net BIN11: now reaches U10.17 (BIN1)
- net STBY1: now reaches U10.19 (STBY)
- net AIN11: now reaches U10.21 (AIN1)
- net AIN21: now reaches U10.22 (AIN2)
- net PWMA1: now reaches U10.23 (PWMA)
- net PWMB0: now reaches U9.15 (PWMB)
- net BIN20: now reaches U9.16 (BIN2)
- net BIN10: now reaches U9.17 (BIN1)
- net STBY0: now reaches U9.19 (STBY)
- net AIN10: now reaches U9.21 (AIN1)
- net AIN20: now reaches U9.22 (AIN2)
- net PWMA0: now reaches U9.23 (PWMA)
Changed lines of the file:
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@@
+    (stroke (width 0) (type default))
+  )
+  (wire (pts (xy 77.47 80.01) (xy 83.82 80.01))
     (stroke (width 0) (type default))
   )
@@
     (stroke (width 0) (type default))
   )
+  (wire (pts (xy 173.99 95.25) (xy 180.34 95.25))
+    (stroke (width 0) (type default))
+  )
   (wire (pts (xy 212.09 78.74) (xy 212.09 80.01))
     (stroke (width 0) (type default))
   )
+  (wire (pts (xy 77.47 92.71) (xy 83.82 92.71))
+    (stroke (width 0) (type default))
+  )
   (wire (pts (xy 212.09 76.2) (xy 217.17 76.2))
     (stroke (width 0) (type default))
@@
     (stroke (width 0) (type default))
   )
+  (wire (pts (xy 77.47 74.93) (xy 83.82 74.93))
+    (stroke (width 0) (type default))
+  )
+  (wire (pts (xy 173.99 87.63) (xy 180.34 87.63))
+    (stroke (width 0) (type default))
+  )
   (wire (pts (xy 120.65 78.74) (xy 115.57 78.74))
     (stroke (width 0) (type default))
@@
     (stroke (width 0) (type default))
   )
+  (wire (pts (xy 173.99 92.71) (xy 180.34 92.71))
+    (stroke (width 0) (type default))
+  )
+  (wire (pts (xy 173.99 80.01) (xy 180.34 80.01))
+    (stroke (width 0) (type default))
+  )
   (wire (pts (xy 115.57 91.44) (xy 115.57 92.71))
     (stroke (width 0) (type default))
@@
     (stroke (width 0) (type default))
   )
+  (wire (pts (xy 77.47 82.55) (xy 83.82 82.55))
+    (stroke (width 0) (type default))
+  )
   (wire (pts (xy 212.09 74.93) (xy 212.09 76.2))
     (stroke (width 0) (type default))
@@
     (stroke (width 0) (type default))
   )
+  (wire (pts (xy 77.47 95.25) (xy 83.82 95.25))
+    (stroke (width 0) (type default))
+  )
   (wire (pts (xy 106.68 111.76) (xy 101.6 111.76))
     (stroke (width 0) (type default))
@@
     (stroke (width 0) (type default))
   )
+  (wire (pts (xy 173.99 82.55) (xy 180.34 82.55))
+    (stroke (width 0) (type default))
+  )
   (wire (pts (xy 212.09 91.44) (xy 212.09 92.71))
     (stroke (width 0) (type default))
@@
     (stroke (width 0) (type default))
   )
+  (wire (pts (xy 77.47 90.17) (xy 83.82 90.17))
+    (stroke (width 0) (type default))
+  )
   (wire (pts (xy 217.17 91.44) (xy 212.09 91.44))
     (stroke (width 0) (type default))
@@
     (stroke (width 0) (type default))
   )
+  (wire (pts (xy 173.99 74.93) (xy 180.34 74.93))
+    (stroke (width 0) (type default))
+  )
+  (wire (pts (xy 77.47 87.63) (xy 83.82 87.63))
+    (stroke (width 0) (type default))
+  )
   (wire (pts (xy 91.44 57.15) (xy 91.44 59.69))
     (stroke (width 0) (type default))
@@
     (stroke (width 0) (type default))
   )
+  (wire (pts (xy 173.99 90.17) (xy 180.34 90.17))
+    (stroke (width 0) (type default))
+  )
+  (label "AIN21" (at 173.99 90.17 0) (fields_autoplaced)
+    (effects (font (size 1.27 1.27)) (justify left bottom))
+  )
+  (label "BIN21" (at 173.99 95.25 0) (fields_autoplaced)
+    (effects (font (size 1.27 1.27)) (justify left bottom))
+  )
+  (label "BIN11" (at 173.99 92.71 0) (fields_autoplaced)
+    (effects (font (size 1.27 1.27)) (justify left bottom))
+  )
+  (label "PWMA1" (at 173.99 80.01 0) (fields_autoplaced)
+    (effects (font (size 1.27 1.27)) (justify left bottom))
+  )
+  (label "STBY0" (at 77.47 74.93 0) (fields_autoplaced)
+    (effects (font (size 1.27 1.27)) (justify left bottom))
+  )
+  (label "PWMB1" (at 173.99 82.55 0) (fields_autoplaced)
+    (effects (font (size 1.27 1.27)) (justify left bottom))
+  )
+  (label "PWMB0" (at 77.47 82.55 0) (fields_autoplaced)
+    (effects (font (size 1.27 1.27)) (justify left bottom))
+  )
+  (label "AIN20" (at 77.47 90.17 0) (fields_autoplaced)
+    (effects (font (size 1.27 1.27)) (justify left bottom))
+  )
+  (label "BIN20" (at 77.47 95.25 0) (fields_autoplaced)
+    (effects (font (size 1.27 1.27)) (justify left bottom))
+  )
+  (label "PWMA0" (at 77.47 80.01 0) (fields_autoplaced)
+    (effects (font (size 1.27 1.27)) (justify left bottom))
+  )
+  (label "BIN10" (at 77.47 92.71 0) (fields_autoplaced)
+    (effects (font (size 1.27 1.27)) (justify left bottom))
+  )
+  (label "AIN10" (at 77.47 87.63 0) (fields_autoplaced)
+    (effects (font (size 1.27 1.27)) (justify left bottom))
+  )
+  (label "AIN11" (at 173.99 87.63 0) (fields_autoplaced)
+    (effects (font (size 1.27 1.27)) (justify left bottom))
+  )
+  (label "STBY1" (at 173.99 74.93 0) (fields_autoplaced)
+    (effects (font (size 1.27 1.27)) (justify left bottom))
+  )
   (symbol (lib_id "Connector:Conn_01x02_Socket") (at 222.25 88.9 0) (unit 1)

Commit message: 2023/3/29
Parts:
- removed J2, J3, J4, J5: Conn_01x02_Socket, symbol Connector:Conn_01x02_Socket
- removed U10, U9: TB6612FNG, Package_SO:SSOP-24_5.3x8.2mm_P0.65mm, symbol Driver_Motor:TB6612FNG
- added C17 (x3): 10uF, Capacitor_SMD:CP_Elec_4x5.4, symbol Device:C_Polarized
- added C5 (x3): 104, Capacitor_SMD:C_0402_1005Metric, symbol Device:C
- added J4, J5, J6: Conn_01x02, Connector_JST:JST_XH_B1B-XH-AM_1x01_P2.50mm_Vertical, symbol Connector_Generic:Conn_01x02
- added U6, U7, U8: DRV8820DSG, Package_SON:WSON-8-1EP_2x2mm_P0.5mm_EP0.9x1.6mm, symbol Driver_Motor:DRV8220DSG
Connections:
- net +12V: now also C17.1, C17.1, C17.1, C5.1, C5.1, C5.1, U6.1 (VM), U7.1 (VM), U8.1 (VM)
- net GND: now also C17.2, C17.2, C17.2, C5.2, C5.2, C5.2, U6.4 (GND), U6.9 (GND), U7.4 (GND), U7.9 (GND), U8.4 (GND), U8.9 (GND)
- new net: J6.1 (Pin_1), U8.2 (OUT1)
- new net: J6.2 (Pin_2), U8.3 (OUT2)
- new net: J5.1 (Pin_1), U7.2 (OUT1)
- new net: J5.2 (Pin_2), U7.3 (OUT2)
- new net: J4.1 (Pin_1), U6.2 (OUT1)
- new net: J4.2 (Pin_2), U6.3 (OUT2)
- new net +3V3: U6.7 (MODE), U7.6 (IN1/PH), U7.7 (MODE), U8.6 (IN1/PH), U8.7 (MODE)
- new net AEN: U6.5 (IN2/EN)
- new net APH: U6.6 (IN1/PH)
- new net ASLEEP: U6.8 (~{SLEEP})
- new net BEN: U7.5 (IN2/EN)
- new net BSLEEP: U7.8 (~{SLEEP})
- new net CEN: U8.5 (IN2/EN)
- new net CSLEEP: U8.8 (~{SLEEP})

Commit message: nm
Parts:
- J4, J5, J6: footprint Connector_JST:JST_XH_B1B-XH-AM_1x01_P2.50mm_Vertical -> Connector_JST:JST_XH_B2B-XH-A_1x02_P2.50mm_Vertical
Changed lines of the file:
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@@
       (effects (font (size 1.27 1.27)) (justify left))
     )
-    (property "Footprint" "Connector_JST:JST_XH_B1B-XH-AM_1x01_P2.50mm_Vertical" (at 87.63 121.92 0)
+    (property "Footprint" "Connector_JST:JST_XH_B2B-XH-A_1x02_P2.50mm_Vertical" (at 87.63 121.92 0)
       (effects (font (size 1.27 1.27)) hide)
     )
@@
   (symbol (lib_id "power:GND") (at 107.95 38.1 0) (unit 1)
     (in_bom yes) (on_board yes) (dnp no) (fields_autoplaced)
-    (property "Reference" "#PWR050" (at 107.95 44.45 0)
+    (property "Reference" "#PWR047" (at 107.95 44.45 0)
       (effects (font (size 1.27 1.27)) hide)
     )
@@
       (project "Warehouse-on-STM32"
         (path "/2599b9a9-6312-402b-9c24-1e87744a4c70/99bb5e8e-3124-4586-a004-2ab84cf92f19"
-          (reference "#PWR050") (unit 1)
+          (reference "#PWR047") (unit 1)
         )
       )
@@
   (symbol (lib_id "power:GND") (at 107.95 120.65 0) (unit 1)
     (in_bom yes) (on_board yes) (dnp no) (fields_autoplaced)
-    (property "Reference" "#PWR052" (at 107.95 127 0)
+    (property "Reference" "#PWR049" (at 107.95 127 0)
       (effects (font (size 1.27 1.27)) hide)
     )
@@
       (project "Warehouse-on-STM32"
         (path "/2599b9a9-6312-402b-9c24-1e87744a4c70/99bb5e8e-3124-4586-a004-2ab84cf92f19"
-          (reference "#PWR052") (unit 1)
+          (reference "#PWR049") (unit 1)
         )
       )
@@
   (symbol (lib_id "power:GND") (at 107.95 80.01 0) (unit 1)
     (in_bom yes) (on_board yes) (dnp no) (fields_autoplaced)
-    (property "Reference" "#PWR051" (at 107.95 86.36 0)
+    (property "Reference" "#PWR048" (at 107.95 86.36 0)
       (effects (font (size 1.27 1.27)) hide)
     )
@@
       (project "Warehouse-on-STM32"
         (path "/2599b9a9-6312-402b-9c24-1e87744a4c70/99bb5e8e-3124-4586-a004-2ab84cf92f19"
-          (reference "#PWR051") (unit 1)
+          (reference "#PWR048") (unit 1)
         )
       )
@@
       (effects (font (size 1.27 1.27)) (justify left))
     )
-    (property "Footprint" "Connector_JST:JST_XH_B1B-XH-AM_1x01_P2.50mm_Vertical" (at 87.63 39.37 0)
+    (property "Footprint" "Connector_JST:JST_XH_B2B-XH-A_1x02_P2.50mm_Vertical" (at 87.63 39.37 0)
       (effects (font (size 1.27 1.27)) hide)
     )
@@
         )
         (path "/2599b9a9-6312-402b-9c24-1e87744a4c70/99bb5e8e-3124-4586-a004-2ab84cf92f19"
-          (reference "C29") (unit 1)
+          (reference "C28") (unit 1)
         )
       )
@@
   (symbol (lib_id "power:GND") (at 69.85 54.61 0) (unit 1)
     (in_bom yes) (on_board yes) (dnp no) (fields_autoplaced)
-    (property "Reference" "#PWR045" (at 69.85 60.96 0)
+    (property "Reference" "#PWR042" (at 69.85 60.96 0)
       (effects (font (size 1.27 1.27)) hide)
     )
@@
       (project "Warehouse-on-STM32"
         (path "/2599b9a9-6312-402b-9c24-1e87744a4c70/99bb5e8e-3124-4586-a004-2ab84cf92f19"
-          (reference "#PWR045") (unit 1)
+          (reference "#PWR042") (unit 1)
         )
       )
@@
   (symbol (lib_id "power:+12V") (at 69.85 67.31 0) (unit 1)
     (in_bom yes) (on_board yes) (dnp no) (fields_autoplaced)
-    (property "Reference" "#PWR046" (at 69.85 71.12 0)
+    (property "Reference" "#PWR043" (at 69.85 71.12 0)
       (effects (font (size 1.27 1.27)) hide)
     )
@@
       (project "Warehouse-on-STM32"
         (path "/2599b9a9-6312-402b-9c24-1e87744a4c70/99bb5e8e-3124-4586-a004-2ab84cf92f19"
-          (reference "#PWR046") (unit 1)
+          (reference "#PWR043") (unit 1)
         )
       )
@@
         )
         (path "/2599b9a9-6312-402b-9c24-1e87744a4c70/99bb5e8e-3124-4586-a004-2ab84cf92f19"
-          (reference "C26") (unit 1)
+          (reference "C25") (unit 1)
         )
       )
@@
         )
         (path "/2599b9a9-6312-402b-9c24-1e87744a4c70/99bb5e8e-3124-4586-a004-2ab84cf92f19"
-          (reference "#PWR043") (unit 1)
+          (reference "#PWR040") (unit 1)
         )
       )
@@
         )
         (path "/2599b9a9-6312-402b-9c24-1e87744a4c70/99bb5e8e-3124-4586-a004-2ab84cf92f19"
-          (reference "C27") (unit 1)
+          (reference "C26") (unit 1)
         )
       )
@@
         )
         (path "/2599b9a9-6312-402b-9c24-1e87744a4c70/99bb5e8e-3124-4586-a004-2ab84cf92f19"
-          (reference "C28") (unit 1)
+          (reference "C27") (unit 1)
         )
       )
@@
         )
         (path "/2599b9a9-6312-402b-9c24-1e87744a4c70/99bb5e8e-3124-4586-a004-2ab84cf92f19"
-          (reference "#PWR042") (unit 1)
+          (reference "#PWR039") (unit 1)
         )
       )
@@
         )
         (path "/2599b9a9-6312-402b-9c24-1e87744a4c70/99bb5e8e-3124-4586-a004-2ab84cf92f19"
-          (reference "C25") (unit 1)
+          (reference "C24") (unit 1)
         )
       )
@@
         )
         (path "/2599b9a9-6312-402b-9c24-1e87744a4c70/99bb5e8e-3124-4586-a004-2ab84cf92f19"
-          (reference "C30") (unit 1)
+          (reference "C29") (unit 1)
         )
       )
@@
   (symbol (lib_id "power:+12V") (at 69.85 25.4 0) (unit 1)
     (in_bom yes) (on_board yes) (dnp no) (fields_autoplaced)
-    (property "Reference" "#PWR044" (at 69.85 29.21 0)
+    (property "Reference" "#PWR041" (at 69.85 29.21 0)
       (effects (font (size 1.27 1.27)) hide)
     )
@@
       (project "Warehouse-on-STM32"
         (path "/2599b9a9-6312-402b-9c24-1e87744a4c70/99bb5e8e-3124-4586-a004-2ab84cf92f19"
+          (reference "#PWR041") (unit 1)
+        )
+      )
+    )
+  )
+  (symbol (lib_id "power:GND") (at 69.85 96.52 0) (unit 1)
+    (in_bom yes) (on_board yes) (dnp no) (fields_autoplaced)
+    (property "Reference" "#PWR044" (at 69.85 102.87 0)
+      (effects (font (size 1.27 1.27)) hide)
+    )
+    (property "Value" "GND" (at 69.85 101.6 0)
+      (effects (font (size 1.27 1.27)))
+    )
+    (property "Footprint" "" (at 69.85 96.52 0)
+      (effects (font (size 1.27 1.27)) hide)
+    )
+    (property "Datasheet" "" (at 69.85 96.52 0)
+      (effects (font (size 1.27 1.27)) hide)
+    )
+    (pin "1")
+    (instances
+      (project "Warehouse-on-STM32"
+        (path "/2599b9a9-6312-402b-9c24-1e87744a4c70/99bb5e8e-3124-4586-a004-2ab84cf92f19"
           (reference "#PWR044") (unit 1)
-        )
-      )
-    )
-  )
-  (symbol (lib_id "power:GND") (at 69.85 96.52 0) (unit 1)
-    (in_bom yes) (on_board yes) (dnp no) (fields_autoplaced)
-    (property "Reference" "#PWR047" (at 69.85 102.87 0)
-      (effects (font (size 1.27 1.27)) hide)
-    )
-    (property "Value" "GND" (at 69.85 101.6 0)
-      (effects (font (size 1.27 1.27)))
-    )
-    (property "Footprint" "" (at 69.85 96.52 0)
-      (effects (font (size 1.27 1.27)) hide)
-    )
-    (property "Datasheet" "" (at 69.85 96.52 0)
-      (effects (font (size 1.27 1.27)) hide)
-    )
-    (pin "1")
-    (instances
-      (project "Warehouse-on-STM32"
-        (path "/2599b9a9-6312-402b-9c24-1e87744a4c70/99bb5e8e-3124-4586-a004-2ab84cf92f19"
-          (reference "#PWR047") (unit 1)
         )
       )
@@
         )
         (path "/2599b9a9-6312-402b-9c24-1e87744a4c70/99bb5e8e-3124-4586-a004-2ab84cf92f19"
-          (reference "#PWR041") (unit 1)
+          (reference "#PWR038") (unit 1)
         )
       )
@@
   (symbol (lib_id "power:GND") (at 69.85 137.16 0) (unit 1)
     (in_bom yes) (on_board yes) (dnp no) (fields_autoplaced)
-    (property "Reference" "#PWR049" (at 69.85 143.51 0)
+    (property "Reference" "#PWR046" (at 69.85 143.51 0)
       (effects (font (size 1.27 1.27)) hide)
     )
@@
       (project "Warehouse-on-STM32"
         (path "/2599b9a9-6312-402b-9c24-1e87744a4c70/99bb5e8e-3124-4586-a004-2ab84cf92f19"
-          (reference "#PWR049") (unit 1)
+          (reference "#PWR046") (unit 1)
         )
       )
@@
       (effects (font (size 1.27 1.27)) (justify left))
     )
-    (property "Footprint" "Connector_JST:JST_XH_B1B-XH-AM_1x01_P2.50mm_Vertical" (at 87.63 81.28 0)
+    (property "Footprint" "Connector_JST:JST_XH_B2B-XH-A_1x02_P2.50mm_Vertical" (at 87.63 81.28 0)
       (effects (font (size 1.27 1.27)) hide)
     )
@@
   (symbol (lib_id "power:+12V") (at 69.85 107.95 0) (unit 1)
     (in_bom yes) (on_board yes) (dnp no) (fields_autoplaced)
-    (property "Reference" "#PWR048" (at 69.85 111.76 0)
+    (property "Reference" "#PWR045" (at 69.85 111.76 0)
       (effects (font (size 1.27 1.27)) hide)
     )
@@
       (project "Warehouse-on-STM32"
         (path "/2599b9a9-6312-402b-9c24-1e87744a4c70/99bb5e8e-3124-4586-a004-2ab84cf92f19"
-          (reference "#PWR048") (unit 1)
-        )
-      )
+          (reference "#PWR045") (unit 1)
+        )
+      )

Commit message: nm
Parts:
- removed C17 (x3): 10uF, Capacitor_SMD:CP_Elec_4x5.4, symbol Device:C_Polarized
- removed C5 (x3): 104, Capacitor_SMD:C_0402_1005Metric, symbol Device:C
- added C14 (x3): 104, Capacitor_SMD:C_0402_1005Metric, symbol Device:C_Small
- added C14 (x3): 10uF, Capacitor_SMD:C_0201_0603Metric, symbol Device:C_Small
- renumbered U6 to U4, U7 to U5, U8 to U6
Connections:
- net +12V: now also C14.1, C14.1, C14.1, C14.1, C14.1, C14.1
- net GND: now also C14.2, C14.2, C14.2, C14.2, C14.2, C14.2
