File: Hardware/驱动模块.kicad_sch (KiCad schematic)
At the start: 12 parts, among them J4 Conn_01x02, J5 Conn_01x02, J6 Conn_01x02, U4 DRV8820DSG, U5 DRV8820DSG, U6 DRV8820DSG

Commit message: 修改了电机驱动芯片旁的电容封装为0603
Parts:
- C14: footprint Capacitor_SMD:C_0201_0603Metric -> Capacitor_SMD:C_0603_1608Metric
- renumbered J4 to J5, J5 to J6, J6 to J7
Changed lines of the file:
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@@
   (symbol (lib_id "Connector_Generic:Conn_01x02") (at 87.63 121.92 0) (unit 1)
     (in_bom yes) (on_board yes) (dnp no) (fields_autoplaced)
-    (property "Reference" "J6" (at 90.17 122.555 0)
+    (property "Reference" "J7" (at 90.17 122.555 0)
       (effects (font (size 1.27 1.27)) (justify left))
     )
@@
       (project "Warehouse-on-STM32"
         (path "/2599b9a9-6312-402b-9c24-1e87744a4c70/99bb5e8e-3124-4586-a004-2ab84cf92f19"
-          (reference "J6") (unit 1)
+          (reference "J7") (unit 1)
         )
       )
@@
   (symbol (lib_id "power:GND") (at 107.95 38.1 0) (unit 1)
     (in_bom yes) (on_board yes) (dnp no) (fields_autoplaced)
-    (property "Reference" "#PWR049" (at 107.95 44.45 0)
+    (property "Reference" "#PWR052" (at 107.95 44.45 0)
       (effects (font (size 1.27 1.27)) hide)
     )
@@
       (project "Warehouse-on-STM32"
         (path "/2599b9a9-6312-402b-9c24-1e87744a4c70/99bb5e8e-3124-4586-a004-2ab84cf92f19"
-          (reference "#PWR049") (unit 1)
+          (reference "#PWR052") (unit 1)
         )
       )
@@
   (symbol (lib_id "Connector_Generic:Conn_01x02") (at 87.63 39.37 0) (unit 1)
     (in_bom yes) (on_board yes) (dnp no) (fields_autoplaced)
-    (property "Reference" "J4" (at 90.17 40.005 0)
+    (property "Reference" "J5" (at 90.17 40.005 0)
       (effects (font (size 1.27 1.27)) (justify left))
     )
@@
       (project "Warehouse-on-STM32"
         (path "/2599b9a9-6312-402b-9c24-1e87744a4c70/99bb5e8e-3124-4586-a004-2ab84cf92f19"
-          (reference "J4") (unit 1)
+          (reference "J5") (unit 1)
         )
       )
@@
       (effects (font (size 1.27 1.27)) (justify left))
     )
-    (property "Footprint" "Capacitor_SMD:C_0201_0603Metric" (at 96.52 73.66 0)
+    (property "Footprint" "Capacitor_SMD:C_0603_1608Metric" (at 96.52 73.66 0)
       (effects (font (size 1.27 1.27)) hide)
     )
@@
   (symbol (lib_id "power:GND") (at 69.85 54.61 0) (unit 1)
     (in_bom yes) (on_board yes) (dnp no) (fields_autoplaced)
-    (property "Reference" "#PWR044" (at 69.85 60.96 0)
+    (property "Reference" "#PWR047" (at 69.85 60.96 0)
       (effects (font (size 1.27 1.27)) hide)
     )
@@
       (project "Warehouse-on-STM32"
         (path "/2599b9a9-6312-402b-9c24-1e87744a4c70/99bb5e8e-3124-4586-a004-2ab84cf92f19"
-          (reference "#PWR044") (unit 1)
+          (reference "#PWR047") (unit 1)
         )
       )
@@
   (symbol (lib_id "power:+12V") (at 69.85 67.31 0) (unit 1)
     (in_bom yes) (on_board yes) (dnp no) (fields_autoplaced)
-    (property "Reference" "#PWR045" (at 69.85 71.12 0)
+    (property "Reference" "#PWR048" (at 69.85 71.12 0)
       (effects (font (size 1.27 1.27)) hide)
     )
@@
       (project "Warehouse-on-STM32"
         (path "/2599b9a9-6312-402b-9c24-1e87744a4c70/99bb5e8e-3124-4586-a004-2ab84cf92f19"
-          (reference "#PWR045") (unit 1)
+          (reference "#PWR048") (unit 1)
         )
       )
@@
   (symbol (lib_id "power:GND") (at 107.95 80.01 0) (unit 1)
     (in_bom yes) (on_board yes) (dnp no) (fields_autoplaced)
-    (property "Reference" "#PWR050" (at 107.95 86.36 0)
+    (property "Reference" "#PWR053" (at 107.95 86.36 0)
       (effects (font (size 1.27 1.27)) hide)
     )
@@
       (project "Warehouse-on-STM32"
         (path "/2599b9a9-6312-402b-9c24-1e87744a4c70/99bb5e8e-3124-4586-a004-2ab84cf92f19"
-          (reference "#PWR050") (unit 1)
+          (reference "#PWR053") (unit 1)
         )
       )
@@
       (effects (font (size 1.27 1.27)) (justify left))
     )
-    (property "Footprint" "Capacitor_SMD:C_0201_0603Metric" (at 96.52 31.75 0)
+    (property "Footprint" "Capacitor_SMD:C_0603_1608Metric" (at 96.52 31.75 0)
       (effects (font (size 1.27 1.27)) hide)
     )
@@
         )
         (path "/2599b9a9-6312-402b-9c24-1e87744a4c70/99bb5e8e-3124-4586-a004-2ab84cf92f19"
-          (reference "#PWR042") (unit 1)
+          (reference "#PWR045") (unit 1)
         )
       )
@@
         )
         (path "/2599b9a9-6312-402b-9c24-1e87744a4c70/99bb5e8e-3124-4586-a004-2ab84cf92f19"
-          (reference "#PWR041") (unit 1)
+          (reference "#PWR044") (unit 1)
         )
       )
@@
       (effects (font (size 1.27 1.27)) (justify left))
     )
-    (property "Footprint" "Capacitor_SMD:C_0201_0603Metric" (at 96.52 114.3 0)
+    (property "Footprint" "Capacitor_SMD:C_0603_1608Metric" (at 96.52 114.3 0)
       (effects (font (size 1.27 1.27)) hide)
     )
@@
   (symbol (lib_id "power:GND") (at 107.95 120.65 0) (unit 1)
     (in_bom yes) (on_board yes) (dnp no) (fields_autoplaced)
-    (property "Reference" "#PWR051" (at 107.95 127 0)
+    (property "Reference" "#PWR054" (at 107.95 127 0)
       (effects (font (size 1.27 1.27)) hide)
     )
@@
       (project "Warehouse-on-STM32"
         (path "/2599b9a9-6312-402b-9c24-1e87744a4c70/99bb5e8e-3124-4586-a004-2ab84cf92f19"
-          (reference "#PWR051") (unit 1)
+          (reference "#PWR054") (unit 1)
         )
       )
@@
   (symbol (lib_id "power:+12V") (at 69.85 25.4 0) (unit 1)
     (in_bom yes) (on_board yes) (dnp no) (fields_autoplaced)
-    (property "Reference" "#PWR043" (at 69.85 29.21 0)
+    (property "Reference" "#PWR046" (at 69.85 29.21 0)
       (effects (font (size 1.27 1.27)) hide)
     )
@@
       (project "Warehouse-on-STM32"
         (path "/2599b9a9-6312-402b-9c24-1e87744a4c70/99bb5e8e-3124-4586-a004-2ab84cf92f19"
-          (reference "#PWR043") (unit 1)
+          (reference "#PWR046") (unit 1)
         )
       )
@@
   (symbol (lib_id "power:GND") (at 69.85 96.52 0) (unit 1)
     (in_bom yes) (on_board yes) (dnp no) (fields_autoplaced)
-    (property "Reference" "#PWR046" (at 69.85 102.87 0)
+    (property "Reference" "#PWR049" (at 69.85 102.87 0)
       (effects (font (size 1.27 1.27)) hide)
     )
@@
       (project "Warehouse-on-STM32"
         (path "/2599b9a9-6312-402b-9c24-1e87744a4c70/99bb5e8e-3124-4586-a004-2ab84cf92f19"
-          (reference "#PWR046") (unit 1)
+          (reference "#PWR049") (unit 1)
         )
       )
@@
         )
         (path "/2599b9a9-6312-402b-9c24-1e87744a4c70/99bb5e8e-3124-4586-a004-2ab84cf92f19"
-          (reference "#PWR040") (unit 1)
+          (reference "#PWR043") (unit 1)
         )
       )
@@
   (symbol (lib_id "power:GND") (at 69.85 137.16 0) (unit 1)
     (in_bom yes) (on_board yes) (dnp no) (fields_autoplaced)
-    (property "Reference" "#PWR048" (at 69.85 143.51 0)
+    (property "Reference" "#PWR051" (at 69.85 143.51 0)
       (effects (font (size 1.27 1.27)) hide)
     )
@@
       (project "Warehouse-on-STM32"
         (path "/2599b9a9-6312-402b-9c24-1e87744a4c70/99bb5e8e-3124-4586-a004-2ab84cf92f19"
-          (reference "#PWR048") (unit 1)
+          (reference "#PWR051") (unit 1)
         )
       )
@@
   (symbol (lib_id "Connector_Generic:Conn_01x02") (at 87.63 81.28 0) (unit 1)
     (in_bom yes) (on_board yes) (dnp no) (fields_autoplaced)
-    (property "Reference" "J5" (at 90.17 81.915 0)
+    (property "Reference" "J6" (at 90.17 81.915 0)
       (effects (font (size 1.27 1.27)) (justify left))
     )
@@
       (project "Warehouse-on-STM32"
         (path "/2599b9a9-6312-402b-9c24-1e87744a4c70/99bb5e8e-3124-4586-a004-2ab84cf92f19"
-          (reference "J5") (unit 1)
+          (reference "J6") (unit 1)
         )
       )
@@
   (symbol (lib_id "power:+12V") (at 69.85 107.95 0) (unit 1)
     (in_bom yes) (on_board yes) (dnp no) (fields_autoplaced)
-    (property "Reference" "#PWR047" (at 69.85 111.76 0)
+    (property "Reference" "#PWR050" (at 69.85 111.76 0)
       (effects (font (size 1.27 1.27)) hide)
     )
@@
       (project "Warehouse-on-STM32"
         (path "/2599b9a9-6312-402b-9c24-1e87744a4c70/99bb5e8e-3124-4586-a004-2ab84cf92f19"
-          (reference "#PWR047") (unit 1)
-        )
-      )
+          (reference "#PWR050") (unit 1)
+        )
+      )
